File: OptoBoard.sch (KiCad schematic (older format))
At the start: 15 parts, among them J1 CONN_01X05, J2 CONN_01X06, U1 LTV-847

Commit message: Version 1 complete
Updated schematic and PCB. This is the version that was sent for
manufacture as Version 1.
Parts:
- removed U1: LTV-847, Housings_DIP:DIP-16_W7.62mm, symbol LTV-847
- added U1: ILQ1, Housings_DIP:DIP-16_W7.62mm, symbol ILQ1
- D1, D2, D3, D4: footprint (none) -> LEDs:LED_D3.0mm
- J1: footprint (none) -> Connectors_Terminal_Blocks:TerminalBlock_bornier-5_P5.08mm
- J2: footprint (none) -> Connectors_Terminal_Blocks:TerminalBlock_bornier-6_P5.08mm
- R1, R2, R3, R4, R5, R6, R7, R8: footprint (none) -> Resistors_THT:R_Axial_DIN0204_L3.6mm_D1.6mm_P2.54mm_Vertical
Connections:
- net at D1.1 (K): now also U1.1
- net at J2.1 (P1): now also U1.10, U1.11, U1.14, U1.15
- net at J2.4 (P4), R7.2: now also U1.12
- net at J2.3 (P3), R6.2: now also U1.13
- net at J2.2 (P2), R5.2: now also U1.16
- net at J1.5 (P5): now also U1.2, U1.3, U1.6, U1.7
- net at D2.1 (K): now also U1.4
- net at D3.1 (K): now also U1.5
- net at D4.1 (K): now also U1.8
- net at J2.5 (P5), R8.2: now also U1.9
Other:
- moved on the sheet: R5
Changed lines of the file:
@@
 LIBS:contrib
 LIBS:valves
+LIBS:JacobLib
+LIBS:OptoBoard-cache
 EELAYER 25 0
 EELAYER END
@@
 $EndDescr
 $Comp
-L LTV-847 U1
-U 1 1 5C32B8CE
-P 5650 3350
-F 0 "U1" H 5450 4050 50  0000 L CNN
-F 1 "LTV-847" H 5650 4050 50  0000 L CNN
-F 2 "Housings_DIP:DIP-16_W7.62mm" H 5450 2750 50  0001 L CIN
-F 3 "" H 5650 3250 50  0001 L CNN
-	1    5650 3350
-	1    0    0    -1
-$EndComp
-$Comp
 L R R1
 U 1 1 5C32B954
@@
 F 0 "R1" V 4430 2750 50  0000 C CNN
 F 1 "R" V 4350 2750 50  0000 C CNN
-F 2 "" V 4280 2750 50  0001 C CNN
+F 2 "Resistors_THT:R_Axial_DIN0204_L3.6mm_D1.6mm_P2.54mm_Vertical" V 4280 2750 50  0001 C CNN
 F 3 "" H 4350 2750 50  0001 C CNN
 	1    4350 2750
@@
 F 0 "R2" V 4430 3050 50  0000 C CNN
 F 1 "R" V 4350 3050 50  0000 C CNN
-F 2 "" V 4280 3050 50  0001 C CNN
+F 2 "Resistors_THT:R_Axial_DIN0204_L3.6mm_D1.6mm_P2.54mm_Vertical" V 4280 3050 50  0001 C CNN
 F 3 "" H 4350 3050 50  0001 C CNN
 	1    4350 3050
@@
 F 0 "R3" V 4430 3350 50  0000 C CNN
 F 1 "R" V 4350 3350 50  0000 C CNN
-F 2 "" V 4280 3350 50  0001 C CNN
+F 2 "Resistors_THT:R_Axial_DIN0204_L3.6mm_D1.6mm_P2.54mm_Vertical" V 4280 3350 50  0001 C CNN
 F 3 "" H 4350 3350 50  0001 C CNN
 	1    4350 3350
@@
 F 0 "R4" V 4430 3650 50  0000 C CNN
 F 1 "R" V 4350 3650 50  0000 C CNN
-F 2 "" V 4280 3650 50  0001 C CNN
+F 2 "Resistors_THT:R_Axial_DIN0204_L3.6mm_D1.6mm_P2.54mm_Vertical" V 4280 3650 50  0001 C CNN
 F 3 "" H 4350 3650 50  0001 C CNN
 	1    4350 3650
@@
 L R R5
 U 1 1 5C32BA7A
-P 6750 2950
-F 0 "R5" V 6830 2950 50  0000 C CNN
-F 1 "R" V 6750 2950 50  0000 C CNN
-F 2 "" V 6680 2950 50  0001 C CNN
-F 3 "" H 6750 2950 50  0001 C CNN
-	1    6750 2950
+P 6750 2750
+F 0 "R5" V 6830 2750 50  0000 C CNN
+F 1 "R" V 6750 2750 50  0000 C CNN
+F 2 "Resistors_THT:R_Axial_DIN0204_L3.6mm_D1.6mm_P2.54mm_Vertical" V 6680 2750 50  0001 C CNN
+F 3 "" H 6750 2750 50  0001 C CNN
+	1    6750 2750
 	0    1    1    0
 $EndComp
@@
 F 0 "R6" V 6830 3250 50  0000 C CNN
 F 1 "R" V 6750 3250 50  0000 C CNN
-F 2 "" V 6680 3250 50  0001 C CNN
+F 2 "Resistors_THT:R_Axial_DIN0204_L3.6mm_D1.6mm_P2.54mm_Vertical" V 6680 3250 50  0001 C CNN
 F 3 "" H 6750 3250 50  0001 C CNN
 	1    6750 3250
@@
 F 0 "R7" V 6830 3550 50  0000 C CNN
 F 1 "R" V 6750 3550 50  0000 C CNN
-F 2 "" V 6680 3550 50  0001 C CNN
+F 2 "Resistors_THT:R_Axial_DIN0204_L3.6mm_D1.6mm_P2.54mm_Vertical" V 6680 3550 50  0001 C CNN
 F 3 "" H 6750 3550 50  0001 C CNN
 	1    6750 3550
@@
 F 0 "R8" V 6830 3850 50  0000 C CNN
 F 1 "R" V 6750 3850 50  0000 C CNN
-F 2 "" V 6680 3850 50  0001 C CNN
+F 2 "Resistors_THT:R_Axial_DIN0204_L3.6mm_D1.6mm_P2.54mm_Vertical" V 6680 3850 50  0001 C CNN
 F 3 "" H 6750 3850 50  0001 C CNN
 	1    6750 3850
@@
 F 0 "D1" H 4850 2850 50  0000 C CNN
 F 1 "LED" H 4850 2650 50  0000 C CNN
-F 2 "" H 4850 2750 50  0001 C CNN
+F 2 "LEDs:LED_D3.0mm" H 4850 2750 50  0001 C CNN
 F 3 "" H 4850 2750 50  0001 C CNN
 	1    4850 2750
@@
 F 0 "D2" H 4850 3150 50  0000 C CNN
 F 1 "LED" H 4850 2950 50  0000 C CNN
-F 2 "" H 4850 3050 50  0001 C CNN
+F 2 "LEDs:LED_D3.0mm" H 4850 3050 50  0001 C CNN
 F 3 "" H 4850 3050 50  0001 C CNN
 	1    4850 3050
@@
 F 0 "D3" H 4850 3450 50  0000 C CNN
 F 1 "LED" H 4850 3250 50  0000 C CNN
-F 2 "" H 4850 3350 50  0001 C CNN
+F 2 "LEDs:LED_D3.0mm" H 4850 3350 50  0001 C CNN
 F 3 "" H 4850 3350 50  0001 C CNN
 	1    4850 3350
@@
 F 0 "D4" H 4850 3750 50  0000 C CNN
 F 1 "LED" H 4850 3550 50  0000 C CNN
-F 2 "" H 4850 3650 50  0001 C CNN
+F 2 "LEDs:LED_D3.0mm" H 4850 3650 50  0001 C CNN
 F 3 "" H 4850 3650 50  0001 C CNN
 	1    4850 3650
@@
 F 0 "J1" H 3650 3500 50  0000 C CNN
 F 1 "CONN_01X05" V 3750 3200 50  0000 C CNN
-F 2 "" H 3650 3200 50  0001 C CNN
+F 2 "Connectors_Terminal_Blocks:TerminalBlock_bornier-5_P5.08mm" H 3650 3200 50  0001 C CNN
 F 3 "" H 3650 3200 50  0001 C CNN
 	1    3650 3200
@@
 F 0 "J2" H 6300 2650 50  0000 C CNN
 F 1 "CONN_01X06" V 6400 2300 50  0000 C CNN
-F 2 "" H 6300 2300 50  0001 C CNN
+F 2 "Connectors_Terminal_Blocks:TerminalBlock_bornier-6_P5.08mm" H 6300 2300 50  0001 C CNN
 F 3 "" H 6300 2300 50  0001 C CNN
 	1    6300 2300
@@
 $EndComp
 Wire Wire Line
-	5950 2750 6050 2750
-Wire Wire Line
 	6050 2500 6050 3650
 Wire Wire Line
 	6050 3050 5950 3050
-Wire Wire Line
-	6050 3350 5950 3350
 Connection ~ 6050 3050
 Wire Wire Line
 	6050 3650 5950 3650
-Connection ~ 6050 3350
-Wire Wire Line
-	5950 2950 6600 2950
 Wire Wire Line
 	5950 3250 6600 3250
-Wire Wire Line
-	5950 3550 6600 3550
 Wire Wire Line
 	5950 3850 6600 3850
@@
 Connection ~ 6900 3250
 Wire Wire Line
-	3850 3850 5350 3850
-Wire Wire Line
-	5250 3550 5350 3550
-Connection ~ 5250 3850
-Wire Wire Line
-	5250 3250 5350 3250
-Connection ~ 5250 3550
-Wire Wire Line
-	5250 2950 5350 2950
-Connection ~ 5250 3250
+	5250 2900 5350 2950
 Wire Wire Line
 	5000 2750 5350 2750
 Wire Wire Line
-	5000 3050 5350 3050
-Wire Wire Line
 	5000 3350 5350 3350
 Wire Wire Line
-	5000 3650 5350 3650
-Wire Wire Line
 	4500 3650 4700 3650
 Wire Wire Line
@@
 	4050 3650 4200 3650
 Wire Wire Line
-	3850 3400 3850 3850
-Wire Wire Line
-	6150 2500 6150 2950
-Connection ~ 6150 2950
+	3850 3400 3850 3800
 Wire Wire Line
 	6250 2500 6250 3250
 Connection ~ 6250 3250
 Wire Wire Line
-	6350 2500 6350 3550
-Connection ~ 6350 3550
-Wire Wire Line
 	6450 2500 6450 3850
 Connection ~ 6450 3850
 Wire Wire Line
 	6550 2500 6900 2500
-Connection ~ 6900 2950
 Wire Wire Line
 	6900 2500 6900 3850
@@
 Wire Wire Line
 	5800 2500 5800 2000
-Wire Wire Line
-	5250 2950 5250 3850
-Connection ~ 6050 2750
+$Comp
+L ILQ1 U1
+U 1 1 5C39E0D1
+P 5650 3350
+F 0 "U1" H 5450 4050 50  0000 L CNN
+F 1 "ILQ1" H 5650 4050 50  0000 L CNN
+F 2 "Housings_DIP:DIP-16_W7.62mm" H 5450 2750 50  0001 L CIN
+F 3 "" H 5650 3250 50  0001 L CNN
+	1    5650 3350
+	1    0    0    -1
+$EndComp
+Wire Wire Line
+	5950 2750 6600 2750
+Wire Wire Line
+	5950 2950 6050 2950
+Connection ~ 6050 2950
+Wire Wire Line
+	6150 2500 6150 2750
+Connection ~ 6150 2750
+Wire Wire Line
+	6600 3350 6600 3550
+Wire Wire Line
+	5950 3350 6600 3350
+Wire Wire Line
+	6350 2500 6350 3350
+Connection ~ 6350 3350
+Wire Wire Line
+	5950 3550 6050 3550
+Connection ~ 6050 3550
+Connection ~ 6900 2750
+Wire Wire Line
+	5350 3050 5250 3000
+Connection ~ 5250 3000
+Wire Wire Line
+	5250 3550 5350 3550
+Connection ~ 5250 3550
+Wire Wire Line
+	5250 2900 5250 3800
+Wire Wire Line
+	5250 3800 3850 3800
+Wire Wire Line
+	5350 3650 5250 3650
+Connection ~ 5250 3650
+Wire Wire Line
+	5000 3650 5000 3850
+Wire Wire Line
+	5000 3850 5350 3850
+Wire Wire Line
+	5000 3050 5150 3050
+Wire Wire Line
+	5150 3050 5150 3250
+Wire Wire Line
+	5150 3250 5350 3250
 $EndSCHEMATC
